Commit message: launch file for dual gazebo and rviz setup for the rwd bot - added rviz_rwd.launch.py adapted from example code - many diff ways to write launch files and starting certain nodes vs executing processes can be the difference in what joints are loaded (my case) - modifed imu topic route - added sdf (gazebo) files to load worlds - custom rviz (robot-config.rviz) for loading rwd bot in rviz

File: src/diff_drive_control/urdf/imu.xacro (robot description, xacro)
@@ -20,5 +20,4 @@
                 <box size="0.02 0.02 0.02"/>
             </geometry>
-            <material name="Gazebo/Red"/>
         </visual>
         <inertial>
@@ -34,17 +33,5 @@
             <update_rate>1000</update_rate>
             <visualize>1</visualize>
-            <topic>imu_data</topic>
-            <!-- <plugin name='imu_plugin' filename='libgazebo_ros_imu_sensor.so'>
-                <topicName>imu_data</topicName>
-                <bodyName>imu_sensor_link</bodyName>
-                <updateRateHZ>10.0</updateRateHZ>
-                <gaussianNoise>0.0</gaussianNoise>
-                <xyzOffset>0 0 0</xyzOffset>
-                <rpyOffset>0 0 0</rpyOffset>
-            </plugin>
-            <pose>0 0 0 0 0 0</pose> -->
-            <!-- <ros>
-                <namespace>diff_drive_control</namespace>
-            </ros> -->
+            <topic>imu</topic>
             <plugin
                 filename="gz-sim-imu-system"

File: src/diff_drive_control/urdf/rwd.xacro (robot description, xacro)
@@ -31,10 +31,4 @@
         izz="0.1"/>
     </inertial>
-    <!-- <sensor name="imu_sensor" type="imu">
-      <always_on>1</always_on>
-      <update_rate>1</update_rate>
-      <visualize>true</visualize>
-      <topic>imu</topic>
-    </sensor> -->
   </link>
   <!-- Include the wheel macro -->
@@ -67,4 +61,12 @@
         <state_interface name="velocity"/>
     </joint>
+    <joint name="joint_wheel_fl">
+        <state_interface name="position"/>
+        <state_interface name="velocity"/>
+    </joint>
+    <joint name="joint_wheel_fr">
+        <state_interface name="position"/>
+        <state_interface name="velocity"/>
+    </joint>
   </ros2_control>
   <gazebo>
@@ -73,15 +75,4 @@
         <parameters>$(find diff_drive_control)/config/rwd_diff_controller.yaml</parameters>
     </plugin>
-    <!-- <plugin
-        filename="gz-sim-imu-system"
-        name="gz::sim::systems::Imu">
-        <bodyName>base_link</bodyName>
-        <updateRate>100.0</updateRate>
-        <topicName>imu_data</topicName>
-        <serviceName>imu_service</serviceName>
-        <gaussianNoise>0.1</gaussianNoise>
-        <xyzOffset>0 0 0</xyzOffset>
-        <rpyOffset>0 0 0</rpyOffset>
-    </plugin> -->
   </gazebo>
   <gazebo reference="wheel_fl">
