Commit message: implemented a functional (but in progress) model of imu state estimation - imu only provides linear accel, angular vel data, and the reconstruction of position and heading is quite innacurate - also have odom pose info from gazebo which is constructed from the diff drive kinematics todo: 1. get true pose from gazebo model (validation) 2. use rviz instead of gazebo (seems to be better for motion planning and traj following) 3. implement positional pid after imu/odom sensor fusion 4. implement velocity pid w/ motion profile

File: src/diff_drive_control/urdf/rwd.xacro (robot description, xacro)
@@ -3,9 +3,9 @@
 <!-- USEFUL CONSTANTS -->
 <!-- size = x y z -->
-<xacro:property name="robot_size" value="0.5 0.3 0.1"/>
-<xacro:property name="robot_mass" value="5.0"/>
-<xacro:property name="wheel_x" value="0.18"/>
-<xacro:property name="wheel_y" value="0.13"/>
-<xacro:property name="wheel_z" value="-0.05"/>
+<xacro:property name="robot_size" value="5.0 3.0 1.0"/>
+<xacro:property name="robot_mass" value="50.0"/>
+<xacro:property name="wheel_x" value="1.8"/>
+<xacro:property name="wheel_y" value="1.3"/>
+<xacro:property name="wheel_z" value="-0.5"/>
 <xacro:property name="origin" value="0 0 0"/>
   <link name="base_link">

File: src/robot/urdf/wheel.xacro (robot description, xacro)
@@ -1,6 +1,6 @@
 <?xml version="1.0"?>
 <robot xmlns:xacro="http://ros.org/wiki/xacro" name="wheel">
-<xacro:property name="wheel_len" value="0.02"/>
-<xacro:property name="wheel_rad" value="0.05"/>
+<xacro:property name="wheel_len" value="0.2"/>
+<xacro:property name="wheel_rad" value="0.5"/>
   <xacro:macro name="wheel" params="name parent_link xyz">
     <link name="${name}">
@@ -21,5 +21,6 @@
       </collision>
       <inertial>
-        <mass value="0.2"/>
+      <!-- mass was 0.2 -->
+        <mass value="2"/>
         <origin xyz="0 0 0" rpy="0 0 0"/>
         <inertia

Commit message: [fix] added logging to brain node + smaller robot model

File: src/diff_drive_control/urdf/rwd.xacro (robot description, xacro)
@@ -3,9 +3,9 @@
 <!-- USEFUL CONSTANTS -->
 <!-- size = x y z -->
-<xacro:property name="robot_size" value="5.0 3.0 1.0"/>
-<xacro:property name="robot_mass" value="50.0"/>
-<xacro:property name="wheel_x" value="1.8"/>
-<xacro:property name="wheel_y" value="1.3"/>
-<xacro:property name="wheel_z" value="-0.5"/>
+<xacro:property name="robot_size" value="0.5 0.3 0.1"/>
+<xacro:property name="robot_mass" value="5.0"/>
+<xacro:property name="wheel_x" value=".18"/>
+<xacro:property name="wheel_y" value=".13"/>
+<xacro:property name="wheel_z" value="-0.05"/>
 <xacro:property name="origin" value="0 0 0"/>
   <link name="base_link">

File: src/diff_drive_control/urdf/wheel.xacro (robot description, xacro)
@@ -1,6 +1,6 @@
 <?xml version="1.0"?>
 <robot xmlns:xacro="http://ros.org/wiki/xacro" name="wheel">
-<xacro:property name="wheel_len" value="0.2"/>
-<xacro:property name="wheel_rad" value="0.5"/>
+<xacro:property name="wheel_len" value="0.02"/>
+<xacro:property name="wheel_rad" value="0.05"/>
   <xacro:macro name="wheel" params="name parent_link xyz">
     <link name="${name}">

Commit message: [feat] odom + imu sensor fusion localization node, much better accuracy - localization node publishes fused odom/imu data to /get_pose_est topic - ui displays pose estimate alongside true pose - went from 4 wheels to 2 wheels on robot model bc diffdrivecontroller limited options for wheel offsets, and this fixed the odom localization inaccuracy

File: src/diff_drive_control/urdf/rwd.xacro (robot description, xacro)
@@ -5,5 +5,5 @@
 <xacro:property name="robot_size" value="0.5 0.3 0.1"/>
 <xacro:property name="robot_mass" value="5.0"/>
-<xacro:property name="wheel_x" value=".18"/>
+<xacro:property name="wheel_x" value="0"/>
 <xacro:property name="wheel_y" value=".13"/>
 <xacro:property name="wheel_z" value="-0.05"/>
@@ -35,6 +35,6 @@
   <xacro:include filename="./wheel.xacro"/>
   <!-- Instantiate wheels -->
-  <xacro:wheel name="wheel_fl" parent_link="base_link" xyz="${wheel_x} ${wheel_y} ${wheel_z}"/>
-  <xacro:wheel name="wheel_fr" parent_link="base_link" xyz="${wheel_x} ${-wheel_y} ${wheel_z}"/>
+  <!-- <xacro:wheel name="wheel_fl" parent_link="base_link" xyz="${wheel_x} ${wheel_y} ${wheel_z}"/>
+  <xacro:wheel name="wheel_fr" parent_link="base_link" xyz="${wheel_x} ${-wheel_y} ${wheel_z}"/> -->
   <xacro:wheel name="wheel_rl" parent_link="base_link" xyz="${-wheel_x} ${wheel_y} ${wheel_z}"/>
   <xacro:wheel name="wheel_rr" parent_link="base_link" xyz="${-wheel_x} ${-wheel_y} ${wheel_z}"/>
